Commit message: second commit

File: urdf/Assem1.urdf (robot description, URDF)
Before this commit: robot Assem1, 6 links, 5 joints
Links:
- added link lidar, mass 1e-5; collision box size=0.1 0.1 0.1; visual mesh filename=package://almond_sim/meshes/lidar.dae
Joints:
- added joint lidar_joint: type fixed, parent base_link, child lidar, axis 0 1 0
